File: mouflePower.sch (KiCad schematic (older format))
At the start: 41 parts, among them J1 FTDI, J10 EINK, J11 ANALOG, J2 Antenna, J3 I2C, J4 ICSP, J5 V_MAIN, J6 Relay, J7 SPI, J8 I2C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

Commit message: Add flyback diode
Parts:
- added D2: S1K-13-F, Diode_SMD:D_SMA, symbol D
Connections:
- wire segments 155 -> 157
Changed lines of the file:
@@
 $EndComp
 Wire Wire Line
-	4200 4250 3900 4250
+	3700 4250 4200 4250
 Wire Wire Line
 	3900 4250 3900 4350
@@
 L +VDC #PWR028
 U 1 1 5A9B342C
-P 3900 4150
-F 0 "#PWR028" H 3900 4050 50  0001 C CNN
-F 1 "+VDC" H 3900 4400 50  0000 C CNN
-F 2 "" H 3900 4150 50  0001 C CNN
-F 3 "" H 3900 4150 50  0001 C CNN
-	1    3900 4150
+P 3900 3900
+F 0 "#PWR028" H 3900 3800 50  0001 C CNN
+F 1 "+VDC" H 3900 4150 50  0000 C CNN
+F 2 "" H 3900 3900 50  0001 C CNN
+F 3 "" H 3900 3900 50  0001 C CNN
+	1    3900 3900
 	1    0    0    -1
 $EndComp
@@
 Wire Wire Line
 	9550 3950 10050 3950
+$Comp
+L D D2
+U 1 1 5AA99E09
+P 3700 4100
+F 0 "D2" H 3700 4200 50  0000 C CNN
+F 1 "S1K-13-F" H 3700 4000 50  0000 C CNN
+F 2 "Diode_SMD:D_SMA" H 3700 4100 50  0001 C CNN
+F 3 "https://www.mouser.fr/ProductDetail/Diodes-Incorporated/S1K-13-F?qs=sGAEpiMZZMtbRapU8LlZDwq4z0BECS78WVSD7wbc0LQ%3d" H 3700 4100 50  0001 C CNN
+	1    3700 4100
+	0    1    1    0
+$EndComp
+Wire Wire Line
+	3900 3950 3700 3950
+Connection ~ 3900 4250
+Wire Wire Line
+	3900 3900 3900 4150
+Connection ~ 3900 3950
 $EndSCHEMATC
